File: Hardware/Production/Qwiic_GPIO-Panel.brd (EAGLE design)
At the start: 174 x 174 mm, 1141 parts, among them J13 SMD, J14 PTH, J15 SMD, J19 SMD, J2 SMD, J20 PTH, J21 SMD, J25 SMD, J26 PTH, J27 SMD, J3 PTH, J31 SMD, J32 PTH, J33 SMD, J37 SMD, J38 PTH, J39 SMD, J4 SMD, J43 SMD, J44 PTH, J45 SMD, J49 SMD, J50 PTH, J51 SMD, J55 SMD, J56 PTH, J57 SMD, J61 SMD, J62 PTH, J63 SMD, J67 SMD, J68 PTH, J69 SMD, J7 SMD, J73 SMD, J74 PTH, J75 SMD, J79 SMD, J8 PTH, J80 PTH, J81 SMD, J85 SMD, J86 PTH, J87 SMD, J9 SMD, J91 SMD, J92 PTH, J93 SMD, U1 TCA9534U, U10 TCA9534U, U11 TCA9534U, U12 TCA9534U, U13 TCA9534U, U14 TCA9534U, U15 TCA9534U, U16 TCA9534U, U2 TCA9534U, U3 TCA9534U, U4 TCA9534U, U5 TCA9534U, U6 TCA9534U, U7 TCA9534U, U8 TCA9534U, U9 TCA9534U

Commit message: uploading panel
Parts:
- removed 3V1, 3V10, 3V11, 3V12, 3V13, 3V14, 3V15, 3V16, 3V2, 3V4, 3V6, 3V7, 3V8, JP105, JP114, JP123, JP132, JP141, JP42, JP51, JP60, JP69, JP78, JP87, JP96: JUMPER-SMT_2_NC_TRACE_SILK, SparkFun-Jumpers:SMT-JUMPER_2_NC_TRACE_SILK
- removed C10, C11, C12, C13, C14, C15, C16: 0.1uF, SparkFun-Capacitors:0603
- removed D10, D11, D12, D13, D14, D15, D16: RED, SparkFun-LED:LED-0603
- removed FD19, FD20, FD21, FD22, FD23, FD24, FD25, FD26, FD27, FD28, FD29, FD30, FD31, FD32: FIDUCIAL1X2, SparkFun-Aesthetics:FIDUCIAL-1X2
- removed H19, H20, H21, H22, H23, H24, H25, H26, H27, H28, H29, H30, H31, H32: STAND-OFF, SparkFun-Hardware:STAND-OFF
- removed J73, J75, J79, J81, J85, J87, J91, J93: SMD, SparkX:1X04_1MM_RA
- removed J74, J80, J86, J92: PTH, SparkX:1X04_NO_SILK
- removed J76, J82, J88, J94: (no value), SparkFun-Connectors:1X01_NO_SILK
- removed J77, J78, J83, J84, J89, J90, J95, J96: (no value), SparkFun-Connectors:LATCHTERMINAL-5MM-4
- removed JP100, JP101, JP109, JP110, JP118, JP119, JP127, JP128, JP136, JP137, JP37, JP38, JP46, JP47, JP55, JP56, JP64, JP65, JP73, JP74, JP82, JP83, JP91, JP92: STAND-OFF, SparkFun:STAND-OFF
- removed JP102, JP103, JP111, JP112, JP120, JP121, JP129, JP130, JP138, JP139, JP39, JP40, JP48, JP49, JP57, JP58, JP66, JP67, JP75, JP76, JP84, JP85, JP93, JP94: FIDUCIAL1X2, SparkFun:FIDUCIAL-1X2
- removed JP104, JP113, JP122, JP131, JP140, JP50, JP59, JP68, JP86, JP95: JUMPER-SMT_3_2-NC_TRACE_SILK, SparkFun-Jumpers:SMT-JUMPER_3_2-NC_TRACE_SILK
- removed JP106, JP107, JP108, JP115, JP116, JP117, JP124, JP125, JP126, JP133, JP134, JP135, JP142, JP143, JP144, JP43, JP44, JP45, JP52, JP53, JP54, JP61, JP62, JP63, JP70, JP71, JP72, JP79, JP80, JP81, JP88, JP89, JP90, JP97, JP98, JP99: (no value), SparkFun-Jumpers:SMT-JUMPER_2_NC_TRACE_SILK
- removed R100, R101, R102, R103, R106, R107, R108, R109, R110, R64, R65, R66, R67, R68, R71, R72, R73, R74, R75, R78, R79, R80, R81, R82, R85, R86, R87, R88, R89, R92, R93, R94, R95, R96, R99: 2.2k, SparkFun-Resistors:0603
- removed R104, R111, R69, R76, R83, R90, R97: 10k, SparkFun-Resistors:0603
- removed R105, R112, R70, R77, R84, R91, R98: 1k, SparkFun-Resistors:0603
- removed U$289, U$329, U$369, U$409, U$449, U$489, U$529, U$569, U$609: (no value), buzzard_labels (45):A00
- removed U$290, U$330, U$370, U$410, U$450, U$490, U$530, U$570, U$610: (no value), buzzard_labels (45):A21
- removed U$291, U$331, U$371, U$411, U$451, U$491, U$531, U$571, U$611: (no value), Labels:I_SUPER2_C-()-03
- removed U$292, U$332, U$372, U$412, U$452, U$492, U$532, U$572, U$612: (no value), SparkFun-Aesthetics:QWIIC_6MM
- removed U$293, U$333, U$373, U$413, U$453, U$493, U$533, U$573, U$613: (no value), buzzard_labels (51):SCL0
- removed U$294, U$334, U$374, U$414, U$454, U$494, U$534, U$574, U$614: (no value), buzzard_labels (51):SDA1
- removed U$295, U$325, U$335, U$365, U$375, U$405, U$415, U$445, U$455, U$485, U$495, U$525, U$535, U$565, U$575, U$605, U$615: (no value), buzzard_labels (44):GND4
- removed U$296, U$323, U$336, U$363, U$376, U$403, U$416, U$443, U$456, U$483, U$496, U$523, U$536, U$563, U$576, U$603, U$616: (no value), buzzard_labels (44):3V33
- removed U$297, U$337, U$377, U$417, U$457, U$497, U$537, U$577, U$617: (no value), buzzard_labels (52):#INT0
- removed U$298, U$338, U$378, U$418, U$458, U$498, U$538, U$578, U$618: (no value), buzzard_labels (54):#INT0
- removed U$299, U$339, U$379, U$419, U$459, U$499, U$539, U$579, U$619: (no value), buzzard_labels (60):QWIIC1
- removed U$300, U$340, U$380, U$420, U$460, U$500, U$540, U$580, U$620: (no value), buzzard_labels (61):GPIO1
- removed U$301, U$341, U$381, U$421, U$461, U$501, U$541, U$581, U$621: (no value), buzzard_labels (5):04
- removed U$302, U$342, U$382, U$422, U$462, U$502, U$542, U$582, U$622: (no value), buzzard_labels (5):15
- removed U$303, U$343, U$383, U$423, U$463, U$503, U$543, U$583, U$623: (no value), buzzard_labels (5):20
- removed U$304, U$344, U$384, U$424, U$464, U$504, U$544, U$584, U$624: (no value), buzzard_labels (5):31
- removed U$305, U$345, U$385, U$425, U$465, U$505, U$545, U$585, U$625: (no value), buzzard_labels (5):GND2
- removed U$306, U$346, U$386, U$426, U$466, U$506, U$546, U$586, U$626: (no value), buzzard_labels (5):3V33
- removed U$307, U$347, U$387, U$427, U$467, U$507, U$547, U$587, U$627: (no value), buzzard_labels (62):3V32
- removed U$308, U$348, U$388, U$428, U$468, U$508, U$548, U$588, U$628: (no value), buzzard_labels (62):GND1
- removed U$309, U$310, U$349, U$350, U$389, U$390, U$429, U$430, U$469, U$470, U$509, U$510, U$549, U$550, U$589, U$590, U$629, U$630: (no value), buzzard_labels (66):INT1
- removed U$311, U$312, U$351, U$352, U$391, U$392, U$431, U$432, U$471, U$472, U$511, U$512, U$551, U$552, U$591, U$592, U$631, U$632: (no value), buzzard_labels (66):PWR0
- removed U$313, U$353, U$393, U$433, U$473, U$513, U$553, U$593, U$633: (no value), buzzard_labels (68):____0____1
- removed U$314, U$354, U$394, U$434, U$474, U$514, U$554, U$594, U$634: (no value), buzzard_labels (68):____2____3
- removed U$315, U$355, U$395, U$435, U$475, U$515, U$555, U$595, U$635: (no value), buzzard_labels (68):____3____4
- removed U$316, U$356, U$396, U$436, U$476, U$516, U$556, U$596, U$636: (no value), buzzard_labels (68):_____1____2
- removed U$317, U$318, U$357, U$358, U$397, U$398, U$437, U$438, U$477, U$478, U$517, U$518, U$557, U$558, U$597, U$598, U$637, U$638: (no value), buzzard_labels (68):GND0
- removed U$319, U$320, U$359, U$360, U$399, U$400, U$439, U$440, U$479, U$480, U$519, U$520, U$559, U$560, U$599, U$600, U$639, U$640: (no value), buzzard_labels (71):_3V3_0
- removed U$321, U$322, U$361, U$362, U$401, U$402, U$441, U$442, U$481, U$482, U$521, U$522, U$561, U$562, U$601, U$602: SPARKX-LOGO3, SparkX:SPARKX-SMALL
- removed U$324, U$364, U$404, U$444, U$484, U$524, U$564, U$604: (no value), buzzard_labels (44):A11
- removed U$326, U$366, U$406, U$446, U$486, U$526, U$566, U$606: (no value), buzzard_labels (44):QWIIC_GPIO7
- removed U$327, U$367, U$407, U$447, U$487, U$527, U$567, U$607: (no value), buzzard_labels (44):SCL6
- removed U$328, U$368, U$408, U$448, U$488, U$528, U$568, U$608: (no value), buzzard_labels (44):SDA5
- removed U10, U11, U12, U13, U14, U15, U16: TCA9534U, KevinKuwata_eagle:16SOIC
- added ADR0, ADR1, ADR10, ADR11, ADR12, ADR13, ADR14, ADR15, ADR16, ADR17, ADR18, ADR19, ADR2, ADR20, ADR21, ADR22, ADR23, ADR24, ADR25, ADR26, ADR3, ADR4, ADR5, ADR6, ADR7, ADR8, ADR9, INT, INT1, INT2, INT3, INT4, INT5, INT6, INT7, INT8, PWR1, PWR2, PWR4, PWR5, PWR7, PWR8: JUMPER-SMT_2_NC_TRACE_SILK, SparkFun-Jumpers:SMT-JUMPER_2_NC_TRACE_SILK
- added FRAME1, FRAME2, FRAME3, FRAME4, FRAME5, FRAME6, FRAME7, FRAME8, FRAME9: FRAME-LETTER, SparkFun-Aesthetics:CREATIVE_COMMONS
- added I2C, I2C1, I2C2, I2C4, I2C5, I2C7, I2C8: JUMPER-SMT_3_2-NC_TRACE_SILK, SparkFun-Jumpers:SMT-JUMPER_3_2-NC_TRACE_SILK
- added LOGO17, LOGO21, LOGO25, LOGO29, LOGO33: OSHW-LOGOMINI, SparkFun-Aesthetics:OSHW-LOGO-MINI
- added LOGO18, LOGO22, LOGO26, LOGO30, LOGO34: REVISION, SparkFun-Aesthetics:REVISION
- added LOGO19, LOGO23, LOGO27, LOGO31, LOGO35: SFE_LOGO_NAME_FLAME.1_INCH, SparkFun-Aesthetics:SFE_LOGO_NAME_FLAME_.1
- added LOGO20, LOGO24, LOGO28, LOGO32, LOGO36: SFE_LOGO_FLAME.2_INCH, SparkFun-Aesthetics:SFE_LOGO_FLAME_.2
- J1, J22, J28, J46, J52, J70: device SparkFun-Connectors:1X01_NO_SILK -> SparkFun-Connectors:LATCHTERMINAL-5MM-4
- J10, J34, J58: value (none) -> QWIIC; device SparkFun-Connectors:1X01_NO_SILK -> SparkFun-Connectors:JST04_1MM_RA
- J13, J19, J21, J27, J37, J43, J45, J51, J61, J67, J69: value SMD -> (none); device SparkX:1X04_1MM_RA -> SparkFun-Connectors:LATCHTERMINAL-5MM-4
- J14, J20, J38, J44, J62, J68, J8: value PTH -> (none); device SparkX:1X04_NO_SILK -> SparkFun-Connectors:LATCHTERMINAL-5MM-4
- J15, J31, J39, J55, J63, J7: value SMD -> (none); device SparkX:1X04_1MM_RA -> SparkFun-Connectors:1X01_NO_SILK
- J16, J40, J64: device SparkFun-Connectors:1X01_NO_SILK -> SparkFun-Connectors:1X04_NO_SILK
- J17, J18, J41, J42, J65, J66: value (none) -> QWIIC; device SparkFun-Connectors:LATCHTERMINAL-5MM-4 -> SparkFun-Connectors:JST04_1MM_RA
- J2, J25, J33, J4, J49, J57: value SMD -> QWIIC; device SparkX:1X04_1MM_RA -> SparkFun-Connectors:JST04_1MM_RA
- J23, J47, J71: device SparkFun-Connectors:LATCHTERMINAL-5MM-4 -> SparkFun-Connectors:1X01_NO_SILK
- J24, J48, J72: device SparkFun-Connectors:LATCHTERMINAL-5MM-4 -> SparkFun-Connectors:1X04_NO_SILK
- J26, J3, J50: value PTH -> QWIIC; device SparkX:1X04_NO_SILK -> SparkFun-Connectors:JST04_1MM_RA
- J32, J56: value PTH -> (none); device SparkX:1X04_NO_SILK -> SparkFun-Connectors:1X04_NO_SILK
- J9: value SMD -> (none); device SparkX:1X04_1MM_RA -> SparkFun-Connectors:1X04_NO_SILK
- JP1, JP17, JP18, JP25, JP26, JP34, JP5: value (none) -> STAND-OFF; device SparkFun-Jumpers:SMT-JUMPER_2_NC_TRACE_SILK -> SparkFun:STAND-OFF
- JP10, JP14: value JUMPER-SMT_3_2-NC_TRACE_SILK -> STAND-OFF; device SparkFun-Jumpers:SMT-JUMPER_3_2-NC_TRACE_SILK -> SparkFun:STAND-OFF
- JP11, JP19, JP20, JP28: value STAND-OFF -> FIDUCIAL1X2; device SparkFun:STAND-OFF -> SparkFun:FIDUCIAL-1X2
- JP13, JP21, JP22, JP30: value FIDUCIAL1X2 -> STAND-OFF; device SparkFun:FIDUCIAL-1X2 -> SparkFun:STAND-OFF
- JP15, JP24, JP8: value JUMPER-SMT_2_NC_TRACE_SILK -> FIDUCIAL1X2; device SparkFun-Jumpers:SMT-JUMPER_2_NC_TRACE_SILK -> SparkFun:FIDUCIAL-1X2
- JP16, JP27, JP35, JP36, JP7: value (none) -> FIDUCIAL1X2; device SparkFun-Jumpers:SMT-JUMPER_2_NC_TRACE_SILK -> SparkFun:FIDUCIAL-1X2
- JP23, JP32: value JUMPER-SMT_3_2-NC_TRACE_SILK -> FIDUCIAL1X2; device SparkFun-Jumpers:SMT-JUMPER_3_2-NC_TRACE_SILK -> SparkFun:FIDUCIAL-1X2
- JP33: value JUMPER-SMT_2_NC_TRACE_SILK -> STAND-OFF; device SparkFun-Jumpers:SMT-JUMPER_2_NC_TRACE_SILK -> SparkFun:STAND-OFF
- LOGO10, LOGO14, LOGO2, LOGO6: value OSHW-LOGOMINI -> REVISION; device SparkFun-Aesthetics:OSHW-LOGO-MINI -> SparkFun-Aesthetics:REVISION
- LOGO11, LOGO15, LOGO3, LOGO7: value OSHW-LOGOMINI -> SFE_LOGO_NAME_FLAME.1_INCH; device SparkFun-Aesthetics:OSHW-LOGO-MINI -> SparkFun-Aesthetics:SFE_LOGO_NAME_FLAME_.1
- LOGO12, LOGO16, LOGO4, LOGO8: value OSHW-LOGOMINI -> SFE_LOGO_FLAME.2_INCH; device SparkFun-Aesthetics:OSHW-LOGO-MINI -> SparkFun-Aesthetics:SFE_LOGO_FLAME_.2
- U$1: value SPARKX-LOGO3 -> (none); device SparkX:SPARKX-SMALL -> SparkFun-Buzzard:I2C
- U$100, U$260: device buzzard_labels (61):GPIO1 -> buzzard_labels (44):SCL6
- U$101, U$261: device buzzard_labels (5):04 -> buzzard_labels (44):SDA5
- U$102, U$262: device buzzard_labels (5):15 -> SparkFun-Aesthetics:QWIIC_6MM
- U$103, U$263: device buzzard_labels (5):20 -> buzzard_labels (51):SCL0
- U$104, U$264: device buzzard_labels (5):31 -> buzzard_labels (51):SDA1
- U$105, U$265: device buzzard_labels (5):GND2 -> buzzard_labels (44):GND4
- U$106, U$266: device buzzard_labels (5):3V33 -> buzzard_labels (44):3V33
- U$107, U$267: device buzzard_labels (62):3V32 -> buzzard_labels (52):#INT0
- U$108, U$268: device buzzard_labels (62):GND1 -> buzzard_labels (54):#INT0
- U$109, U$269: device buzzard_labels (66):INT1 -> SparkFun-Buzzard:I2C
- U$11: device buzzard_labels (45):A00 -> output:#ADR2#0
- U$110, U$270: device buzzard_labels (66):INT1 -> output:PWR0
- U$111, U$271: device buzzard_labels (66):PWR0 -> output:#INT#0
- U$112, U$272, U$39: device buzzard_labels (66):PWR0 -> output:#PWR#0
- U$113, U$273: device buzzard_labels (68):____0____1 -> output:20
- U$114, U$274: device buzzard_labels (68):____2____3 -> output:30
- U$115, U$275: device buzzard_labels (68):____3____4 -> output:10
- U$116, U$276: device buzzard_labels (68):_____1____2 -> output:00
- U$117, U$277: device buzzard_labels (68):GND0 -> output:#INT0
- U$118, U$278: device buzzard_labels (68):GND0 -> output:3V30
- U$119, U$279: device buzzard_labels (71):_3V3_0 -> output:3V30
- U$12: device buzzard_labels (45):A21 -> output:#INT#0
- U$120, U$280: device buzzard_labels (71):_3V3_0 -> output:40
- U$121, U$281: value SPARKX-LOGO3 -> (none); device SparkX:SPARKX-SMALL -> output:50
- U$122, U$282: value SPARKX-LOGO3 -> (none); device SparkX:SPARKX-SMALL -> output:60
- U$123, U$283: device buzzard_labels (44):3V33 -> output:70
- U$124, U$284: device buzzard_labels (44):A11 -> output:#GND#0
- U$125, U$285: device buzzard_labels (44):GND4 -> output:#GND#0
- U$126, U$286: device buzzard_labels (44):QWIIC_GPIO7 -> output:#ADR0#0
- U$127, U$287: device buzzard_labels (44):SCL6 -> output:#ADR1#0
- U$128, U$288: device buzzard_labels (44):SDA5 -> output:#ADR2#0
- U$129: device buzzard_labels (45):A00 -> buzzard_labels (44):3V33
- U$130: device buzzard_labels (45):A21 -> buzzard_labels (44):GND4
- U$131: device Labels:I_SUPER2_C-()-03 -> buzzard_labels (44):QWIIC_GPIO7
- U$132: device SparkFun-Aesthetics:QWIIC_6MM -> buzzard_labels (44):SCL6
- U$133: device buzzard_labels (51):SCL0 -> buzzard_labels (44):SDA5
- U$134: device buzzard_labels (51):SDA1 -> SparkFun-Aesthetics:QWIIC_6MM
- U$135: device buzzard_labels (44):GND4 -> buzzard_labels (51):SCL0
- U$136: device buzzard_labels (44):3V33 -> buzzard_labels (51):SDA1
- U$137: device buzzard_labels (52):#INT0 -> buzzard_labels (44):GND4
- U$138: device buzzard_labels (54):#INT0 -> buzzard_labels (44):3V33
- U$139: device buzzard_labels (60):QWIIC1 -> buzzard_labels (52):#INT0
- U$14: device buzzard_labels (44):3V33 -> output:00
- U$140: device buzzard_labels (61):GPIO1 -> buzzard_labels (54):#INT0
- U$141: device buzzard_labels (5):04 -> SparkFun-Buzzard:I2C
- U$142: device buzzard_labels (5):15 -> output:PWR0
- U$143: device buzzard_labels (5):20 -> output:#INT#0
- U$144: device buzzard_labels (5):31 -> output:#PWR#0
- U$145: device buzzard_labels (5):GND2 -> output:20
- U$146: device buzzard_labels (5):3V33 -> output:30
- U$147: device buzzard_labels (62):3V32 -> output:10
- U$148: device buzzard_labels (62):GND1 -> output:00
- U$149: device buzzard_labels (66):INT1 -> output:#INT0
- U$15: device buzzard_labels (44):A11 -> output:#ADR0#0
- U$150, U$30, U$31: device buzzard_labels (66):INT1 -> output:3V30
- U$151: device buzzard_labels (66):PWR0 -> output:3V30
- U$152: device buzzard_labels (66):PWR0 -> output:40
- U$153: device buzzard_labels (68):____0____1 -> output:50
- U$154: device buzzard_labels (68):____2____3 -> output:60
- U$155: device buzzard_labels (68):____3____4 -> output:70
- U$156: device buzzard_labels (68):_____1____2 -> output:#GND#0
- U$157: device buzzard_labels (68):GND0 -> output:#GND#0
- U$158: device buzzard_labels (68):GND0 -> output:#ADR0#0
- U$159: device buzzard_labels (71):_3V3_0 -> output:#ADR1#0
- U$16: device buzzard_labels (44):GND4 -> buzzard_labels (44):3V33
- U$160: device buzzard_labels (71):_3V3_0 -> output:#ADR2#0
- U$161, U$202: value SPARKX-LOGO3 -> (none); device SparkX:SPARKX-SMALL -> buzzard_labels (44):3V33
- U$162, U$201: value SPARKX-LOGO3 -> (none); device SparkX:SPARKX-SMALL -> buzzard_labels (44):GND4
- U$163: device buzzard_labels (44):3V33 -> buzzard_labels (44):QWIIC_GPIO7
- U$164: device buzzard_labels (44):A11 -> buzzard_labels (44):SCL6
- U$165: device buzzard_labels (44):GND4 -> buzzard_labels (44):SDA5
- U$166: device buzzard_labels (44):QWIIC_GPIO7 -> SparkFun-Aesthetics:QWIIC_6MM
- U$167: device buzzard_labels (44):SCL6 -> buzzard_labels (51):SCL0
- U$168: device buzzard_labels (44):SDA5 -> buzzard_labels (51):SDA1
- U$169: device buzzard_labels (45):A00 -> buzzard_labels (44):GND4
- U$17: device buzzard_labels (44):QWIIC_GPIO7 -> buzzard_labels (44):GND4
- U$170: device buzzard_labels (45):A21 -> buzzard_labels (44):3V33
- U$171: device Labels:I_SUPER2_C-()-03 -> buzzard_labels (52):#INT0
- U$172: device SparkFun-Aesthetics:QWIIC_6MM -> buzzard_labels (54):#INT0
- U$173: device buzzard_labels (51):SCL0 -> SparkFun-Buzzard:I2C
- U$174: device buzzard_labels (51):SDA1 -> output:PWR0
- U$175: device buzzard_labels (44):GND4 -> output:#INT#0
- U$176: device buzzard_labels (44):3V33 -> output:#PWR#0
- U$177: device buzzard_labels (52):#INT0 -> output:20
- U$178: device buzzard_labels (54):#INT0 -> output:30
- U$179: device buzzard_labels (60):QWIIC1 -> output:10
- U$18: device buzzard_labels (44):SCL6 -> buzzard_labels (44):QWIIC_GPIO7
- U$180: device buzzard_labels (61):GPIO1 -> output:00
- U$181: device buzzard_labels (5):04 -> output:#INT0
- U$182: device buzzard_labels (5):15 -> output:3V30
- U$183: device buzzard_labels (5):20 -> output:3V30
- U$184: device buzzard_labels (5):31 -> output:40
- U$185: device buzzard_labels (5):GND2 -> output:50
- U$186: device buzzard_labels (5):3V33 -> output:60
- U$187: device buzzard_labels (62):3V32 -> output:70
- U$188: device buzzard_labels (62):GND1 -> output:#GND#0
- U$189: device buzzard_labels (66):INT1 -> output:#GND#0
- U$19: device buzzard_labels (44):SDA5 -> buzzard_labels (44):SCL6
- U$190: device buzzard_labels (66):INT1 -> output:#ADR0#0
- U$191: device buzzard_labels (66):PWR0 -> output:#ADR1#0
- U$192: device buzzard_labels (66):PWR0 -> output:#ADR2#0
- U$193: device buzzard_labels (68):____0____1 -> buzzard_labels (44):3V33
- U$194: device buzzard_labels (68):____2____3 -> buzzard_labels (44):GND4
- U$195: device buzzard_labels (68):____3____4 -> buzzard_labels (44):QWIIC_GPIO7
- U$196: device buzzard_labels (68):_____1____2 -> buzzard_labels (44):SCL6
- U$197: device buzzard_labels (68):GND0 -> buzzard_labels (44):SDA5
- U$198: device buzzard_labels (68):GND0 -> SparkFun-Aesthetics:QWIIC_6MM
- U$199: device buzzard_labels (71):_3V3_0 -> buzzard_labels (51):SCL0
- U$2, U$241, U$81: value SPARKX-LOGO3 -> (none); device SparkX:SPARKX-SMALL -> output:20
- U$20: device Labels:I_SUPER2_C-()-03 -> buzzard_labels (44):SDA5
- U$200: device buzzard_labels (71):_3V3_0 -> buzzard_labels (51):SDA1
- U$203: device buzzard_labels (44):3V33 -> buzzard_labels (52):#INT0
- U$204: device buzzard_labels (44):A11 -> buzzard_labels (54):#INT0
- U$205: device buzzard_labels (44):GND4 -> SparkFun-Buzzard:I2C
- U$206: device buzzard_labels (44):QWIIC_GPIO7 -> output:PWR0
- U$207: device buzzard_labels (44):SCL6 -> output:#INT#0
- U$208: device buzzard_labels (44):SDA5 -> output:#PWR#0
- U$209, U$49: device buzzard_labels (45):A00 -> output:20
- U$210, U$50: device buzzard_labels (45):A21 -> output:30
- U$211, U$51: device Labels:I_SUPER2_C-()-03 -> output:10
- U$212, U$52: device SparkFun-Aesthetics:QWIIC_6MM -> output:00
- U$213, U$53: device buzzard_labels (51):SCL0 -> output:#INT0
- U$214, U$54: device buzzard_labels (51):SDA1 -> output:3V30
- U$215, U$55: device buzzard_labels (44):GND4 -> output:3V30
- U$216, U$56: device buzzard_labels (44):3V33 -> output:40
- U$217, U$57: device buzzard_labels (52):#INT0 -> output:50
- U$218, U$58: device buzzard_labels (54):#INT0 -> output:60
- U$219, U$59: device buzzard_labels (60):QWIIC1 -> output:70
- U$220, U$60: device buzzard_labels (61):GPIO1 -> output:#GND#0
- U$221, U$61: device buzzard_labels (5):04 -> output:#GND#0
- U$222, U$62: device buzzard_labels (5):15 -> output:#ADR0#0
- U$223, U$63: device buzzard_labels (5):20 -> output:#ADR1#0
- U$224, U$64: device buzzard_labels (5):31 -> output:#ADR2#0
- U$225, U$65: device buzzard_labels (5):GND2 -> buzzard_labels (44):3V33
- U$226, U$66: device buzzard_labels (5):3V33 -> buzzard_labels (44):GND4
- U$227, U$67: device buzzard_labels (62):3V32 -> buzzard_labels (44):QWIIC_GPIO7
- U$228, U$68: device buzzard_labels (62):GND1 -> buzzard_labels (44):SCL6
- U$229, U$69: device buzzard_labels (66):INT1 -> buzzard_labels (44):SDA5
- U$230, U$70: device buzzard_labels (66):INT1 -> SparkFun-Aesthetics:QWIIC_6MM
- U$231, U$71: device buzzard_labels (66):PWR0 -> buzzard_labels (51):SCL0
- U$232, U$72: device buzzard_labels (66):PWR0 -> buzzard_labels (51):SDA1
- U$233, U$41, U$73: device buzzard_labels (68):____0____1 -> buzzard_labels (44):GND4
- U$234, U$42, U$74: device buzzard_labels (68):____2____3 -> buzzard_labels (44):3V33
- U$235, U$43, U$75: device buzzard_labels (68):____3____4 -> buzzard_labels (52):#INT0
- U$236, U$44, U$76: device buzzard_labels (68):_____1____2 -> buzzard_labels (54):#INT0
- U$237, U$45, U$77: device buzzard_labels (68):GND0 -> SparkFun-Buzzard:I2C
- U$238, U$46, U$78: device buzzard_labels (68):GND0 -> output:PWR0
- U$239, U$47, U$79: device buzzard_labels (71):_3V3_0 -> output:#INT#0
- U$240, U$48, U$80: device buzzard_labels (71):_3V3_0 -> output:#PWR#0
- U$242, U$4, U$82: value SPARKX-LOGO3 -> (none); device SparkX:SPARKX-SMALL -> output:30
- U$243, U$83: device buzzard_labels (44):3V33 -> output:10
- U$244, U$84: device buzzard_labels (44):A11 -> output:00
- U$245, U$85: device buzzard_labels (44):GND4 -> output:#INT0
- U$246, U$86: device buzzard_labels (44):QWIIC_GPIO7 -> output:3V30
- U$247, U$87: device buzzard_labels (44):SCL6 -> output:3V30
- U$248, U$88: device buzzard_labels (44):SDA5 -> output:40
- U$249, U$89: device buzzard_labels (45):A00 -> output:50
- U$250, U$90: device buzzard_labels (45):A21 -> output:60
- U$251, U$91: device Labels:I_SUPER2_C-()-03 -> output:70
- U$252, U$92: device SparkFun-Aesthetics:QWIIC_6MM -> output:#GND#0
- U$253, U$93: device buzzard_labels (51):SCL0 -> output:#GND#0
- U$254, U$94: device buzzard_labels (51):SDA1 -> output:#ADR0#0
- U$255, U$95: device buzzard_labels (44):GND4 -> output:#ADR1#0
- U$256, U$96: device buzzard_labels (44):3V33 -> output:#ADR2#0
- U$257, U$97: device buzzard_labels (52):#INT0 -> buzzard_labels (44):3V33
- U$258, U$98: device buzzard_labels (54):#INT0 -> buzzard_labels (44):GND4
- U$259, U$99: device buzzard_labels (60):QWIIC1 -> buzzard_labels (44):QWIIC_GPIO7
- U$27: device buzzard_labels (62):3V32 -> SparkFun-Aesthetics:QWIIC_6MM
- U$28: device buzzard_labels (62):GND1 -> buzzard_labels (51):SCL0
- U$29: device buzzard_labels (5):15 -> output:#INT0
- U$32: device buzzard_labels (60):QWIIC1 -> output:40
- U$33: device buzzard_labels (5):20 -> output:50
- U$34: device buzzard_labels (5):31 -> output:PWR0
- U$35: device buzzard_labels (5):GND2 -> output:60
- U$36: device buzzard_labels (61):GPIO1 -> buzzard_labels (51):SDA1
- U$37: device buzzard_labels (5):04 -> output:70
- U$38: device buzzard_labels (5):3V33 -> output:#GND#0
- U$40: device buzzard_labels (66):PWR0 -> output:#GND#0
- U$5: device buzzard_labels (44):A11 -> output:#ADR1#0
- U$6: value SPARKX-LOGO3 -> (none); device SparkX:SPARKX-SMALL -> output:10
- U1, U2, U3, U4, U5, U6, U7, U8, U9: value TCA9534U -> TCA9534; device KevinKuwata_eagle:16SOIC -> SparkFun-IC-Conversion:16SOIC
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- renumbered 3V3 to PWR, 3V5 to PWR3, 3V9 to PWR6, JP41 to I2C3, JP77 to I2C6
Connections:
- removed net !INT10: J64.1, R76.1, U11.13
- removed net !INT11: J70.1, R83.1, U12.13
- removed net !INT12: J76.1, R90.1, U13.13
- removed net !INT13: J82.1, R97.1, U14.13
- removed net !INT14: J88.1, R104.1, U15.13
- removed net !INT15: J94.1, R111.1, U16.13
- removed net !INT9: J58.1, R69.1, U10.13
- removed net 3.3V10: 3V11.2, C11.1, J61.2, J62.2, J63.2, J65.4, J66.4, JP95.2, JP96.2, JP97.2, JP98.2, JP99.2, U11.16
- removed net 3.3V11: 3V12.2, C12.1, J67.2, J68.2, J69.2, J71.4, J72.4, JP104.2, JP105.2, JP106.2, JP107.2, JP108.2, U12.16
- removed net 3.3V12: 3V13.2, C13.1, J73.2, J74.2, J75.2, J77.4, J78.4, JP113.2, JP114.2, JP115.2, JP116.2, JP117.2, U13.16
- removed net 3.3V13: 3V14.2, C14.1, J79.2, J80.2, J81.2, J83.4, J84.4, JP122.2, JP123.2, JP124.2, JP125.2, JP126.2, U14.16
- removed net 3.3V14: 3V15.2, C15.1, J85.2, J86.2, J87.2, J89.4, J90.4, JP131.2, JP132.2, JP133.2, JP134.2, JP135.2, U15.16
- removed net 3.3V15: 3V16.2, C16.1, J91.2, J92.2, J93.2, J95.4, J96.4, JP140.2, JP141.2, JP142.2, JP143.2, JP144.2, U16.16
- removed net 3.3V9: 3V10.2, C10.1, J55.2, J56.2, J57.2, J59.4, J60.4, JP86.2, JP87.2, JP88.2, JP89.2, JP90.2, U10.16
- removed net A0: JP1.1, R5.2, U3.1
- removed net A1: JP5.1, R3.2, U3.2
- removed net A10: JP35.1, R25.2, U4.2
- removed net A11: JP36.1, R24.2, U4.3
- removed net A12: JP43.1, R33.2, U5.1
- removed net A13: JP44.1, R32.2, U5.2
- removed net A14: JP45.1, R31.2, U5.3
- removed net A15: JP52.1, R40.2, U6.1
- removed net A16: JP53.1, R39.2, U6.2
- removed net A17: JP54.1, R38.2, U6.3
- removed net A18: JP61.1, R47.2, U7.1
- removed net A19: JP62.1, R46.2, U7.2
- removed net A2: JP7.1, R1.2, U3.3
- removed net A20: JP63.1, R45.2, U7.3
- removed net A21: JP70.1, R54.2, U8.1
- removed net A22: JP71.1, R53.2, U8.2
- removed net A23: JP72.1, R52.2, U8.3
- removed net A24: JP79.1, R61.2, U9.1
- removed net A25: JP80.1, R60.2, U9.2
- removed net A26: JP81.1, R59.2, U9.3
- removed net A27: JP88.1, R68.2, U10.1
- removed net A28: JP89.1, R67.2, U10.2
- removed net A29: JP90.1, R66.2, U10.3
- removed net A3: JP16.1, R12.2, U1.1
- removed net A30: JP97.1, R75.2, U11.1
- removed net A31: JP98.1, R74.2, U11.2
- removed net A32: JP99.1, R73.2, U11.3
- removed net A33: JP106.1, R82.2, U12.1
- removed net A34: JP107.1, R81.2, U12.2
- removed net A35: JP108.1, R80.2, U12.3
- removed net A36: JP115.1, R89.2, U13.1
- removed net A37: JP116.1, R88.2, U13.2
- removed net A38: JP117.1, R87.2, U13.3
- removed net A39: JP124.1, R96.2, U14.1
- removed net A4: JP17.1, R11.2, U1.2
- removed net A40: JP125.1, R95.2, U14.2
- removed net A41: JP126.1, R94.2, U14.3
- removed net A42: JP133.1, R103.2, U15.1
- removed net A43: JP134.1, R102.2, U15.2
- removed net A44: JP135.1, R101.2, U15.3
- removed net A45: JP142.1, R110.2, U16.1
- removed net A46: JP143.1, R109.2, U16.2
- removed net A47: JP144.1, R108.2, U16.3
- removed net A5: JP18.1, R10.2, U1.3
- removed net A6: JP25.1, R19.2, U2.1
- removed net A7: JP26.1, R18.2, U2.2
- removed net A8: JP27.1, R17.2, U2.3
- removed net A9: JP34.1, R26.2, U4.1
- removed net GND10: C11.2, D11.C, J61.1, J62.1, J63.1, J65.1, J66.1, R73.1, R74.1, R75.1, U11.8
- removed net GND11: C12.2, D12.C, J67.1, J68.1, J69.1, J71.1, J72.1, R80.1, R81.1, R82.1, U12.8
- removed net GND12: C13.2, D13.C, J73.1, J74.1, J75.1, J77.1, J78.1, R87.1, R88.1, R89.1, U13.8
- removed net GND13: C14.2, D14.C, J79.1, J80.1, J81.1, J83.1, J84.1, R94.1, R95.1, R96.1, U14.8
- removed net GND14: C15.2, D15.C, J85.1, J86.1, J87.1, J89.1, J90.1, R101.1, R102.1, R103.1, U15.8
- removed net GND15: C16.2, D16.C, J91.1, J92.1, J93.1, J95.1, J96.1, R108.1, R109.1, R110.1, U16.8
- removed net GND9: C10.2, D10.C, J55.1, J56.1, J57.1, J59.1, J60.1, R66.1, R67.1, R68.1, U10.8
- removed net N$28: JP87.1, R69.2
- removed net N$29: D10.A, R70.1
- removed net N$30: 3V10.1, R70.2
- removed net N$31: JP96.1, R76.2
- removed net N$32: D11.A, R77.1
- removed net N$33: 3V11.1, R77.2
- removed net N$34: JP105.1, R83.2
- removed net N$35: D12.A, R84.1
- removed net N$36: 3V12.1, R84.2
- removed net N$37: JP114.1, R90.2
- removed net N$38: D13.A, R91.1
- removed net N$39: 3V13.1, R91.2
- removed net N$40: JP123.1, R97.2
- removed net N$41: D14.A, R98.1
- removed net N$42: 3V14.1, R98.2
- removed net N$43: JP132.1, R104.2
- removed net N$44: D15.A, R105.1
- removed net N$45: 3V15.1, R105.2
- removed net N$46: JP141.1, R111.2
- removed net N$47: D16.A, R112.1
- removed net N$48: 3V16.1, R112.2
- removed net SCL10: J61.4, J62.4, J63.4, R72.1, U11.14
- removed net SCL11: J67.4, J68.4, J69.4, R79.1, U12.14
- removed net SCL12: J73.4, J74.4, J75.4, R86.1, U13.14
- removed net SCL13: J79.4, J80.4, J81.4, R93.1, U14.14
- removed net SCL14: J85.4, J86.4, J87.4, R100.1, U15.14
- removed net SCL15: J91.4, J92.4, J93.4, R107.1, U16.14
- removed net SCL9: J55.4, J56.4, J57.4, R65.1, U10.14
- removed net SCL_PU10: JP86.1, R64.2
- removed net SCL_PU11: JP95.1, R71.2
- removed net SCL_PU12: JP104.1, R78.2
- removed net SCL_PU13: JP113.1, R85.2
- removed net SCL_PU14: JP122.1, R92.2
- removed net SCL_PU15: JP131.1, R99.2
- removed net SCL_PU16: JP140.1, R106.2
- removed net SDA10: J61.3, J62.3, J63.3, R71.1, U11.15
- removed net SDA11: J67.3, J68.3, J69.3, R78.1, U12.15
- removed net SDA12: J73.3, J74.3, J75.3, R85.1, U13.15
- removed net SDA13: J79.3, J80.3, J81.3, R92.1, U14.15
- removed net SDA14: J85.3, J86.3, J87.3, R99.1, U15.15
- removed net SDA15: J91.3, J92.3, J93.3, R106.1, U16.15
- removed net SDA9: J55.3, J56.3, J57.3, R64.1, U10.15
- removed net SDA_PU10: JP86.3, R65.2
- removed net SDA_PU11: JP95.3, R72.2
- removed net SDA_PU12: JP104.3, R79.2
- removed net SDA_PU13: JP113.3, R86.2
- removed net SDA_PU14: JP122.3, R93.2
- removed net SDA_PU15: JP131.3, R100.2
- removed net SDA_PU16: JP140.3, R107.2
- new net ADR0: ADR0.1, R5.2, U3.1
- new net ADR1: ADR1.1, R3.2, U3.2
- new net ADR10: ADR10.1, R25.2, U4.2
- new net ADR11: ADR11.1, R24.2, U4.3
- new net ADR12: ADR12.1, R33.2, U5.1
- new net ADR13: ADR13.1, R32.2, U5.2
- new net ADR14: ADR14.1, R31.2, U5.3
- new net ADR15: ADR15.1, R40.2, U6.1
- new net ADR16: ADR16.1, R39.2, U6.2
- new net ADR17: ADR17.1, R38.2, U6.3
- new net ADR18: ADR18.1, R47.2, U7.1
- new net ADR19: ADR19.1, R46.2, U7.2
- new net ADR2: ADR2.1, R1.2, U3.3
- new net ADR20: ADR20.1, R45.2, U7.3
- new net ADR21: ADR21.1, R54.2, U8.1
- new net ADR22: ADR22.1, R53.2, U8.2
- new net ADR23: ADR23.1, R52.2, U8.3
- new net ADR24: ADR24.1, R61.2, U9.1
- new net ADR25: ADR25.1, R60.2, U9.2
- new net ADR26: ADR26.1, R59.2, U9.3
- new net ADR3: ADR3.1, R12.2, U1.1
- new net ADR4: ADR4.1, R11.2, U1.2
- new net ADR5: ADR5.1, R10.2, U1.3
- new net ADR6: ADR6.1, R19.2, U2.1
- new net ADR7: ADR7.1, R18.2, U2.2
- new net ADR8: ADR8.1, R17.2, U2.3
- new net ADR9: ADR9.1, R26.2, U4.1
- new net P64: J67.2, U9.4
- new net P65: J70.2, U9.6
- new net P66: J70.3, U9.7
- new net P67: J67.3, U9.5
- new net P68: J69.2, U9.9
- new net P69: J69.3, U9.10
- new net P70: J68.2, U9.11
- new net P71: J68.3, U9.12
- net !INT: now also J5.1, J7.1; no longer J1.1
- net !INT1: now also J11.1, J15.1; no longer J10.1
- net !INT2: now also J19.1, J23.1; no longer J16.1
- net !INT3: now also J27.1, J31.1; no longer J22.1
- net !INT4: now also J35.1, J39.1; no longer J28.1
- net !INT5: now also J43.1, J47.1; no longer J34.1
- net !INT6: now also J51.1, J55.1; no longer J40.1
- net !INT7: now also J59.1, J63.1; no longer J46.1
- net !INT8: now also J67.1, J71.1; no longer J52.1
- net 3.3V: now also ADR0.2, ADR1.2, ADR2.2, I2C.2, INT.2, J1.1, J8.4, J9.2; no longer J3.2, J5.4, JP1.2, JP10.2, JP5.2, JP7.2, JP8.2
- net 3.3V1: now also ADR3.2, ADR4.2, ADR5.2, I2C1.2, INT1.2, J10.2, J13.1, J14.4, J16.2, J3.2, PWR1.2; no longer 3V1.2, J11.4, J7.2, J8.2, J9.2, JP14.2, JP15.2, JP16.2, JP17.2, JP18.2
- net 3.3V2: now also ADR6.2, ADR7.2, ADR8.2, I2C2.2, INT2.2, J17.2, J18.2, J20.4, J21.1, J22.4, J24.2, PWR2.2; no longer 3V2.2, J13.2, J14.2, J15.2, J17.4, J18.4, JP23.2, JP24.2, JP25.2, JP26.2, JP27.2
- net 3.3V3: now also ADR10.2, ADR11.2, ADR9.2, I2C3.2, INT3.2, J25.2, J26.2, J28.4, J29.1, J30.4, J32.2, PWR3.2; no longer 3V4.2, J19.2, J20.2, J21.2, J23.4, J24.4, JP32.2, JP33.2, JP34.2, JP35.2, JP36.2
- net 3.3V4: now also ADR12.2, ADR13.2, ADR14.2, I2C4.2, INT4.2, J33.2, J34.2, J36.4, J37.1, J38.4, J40.2, PWR4.2; no longer I2C3.2, J25.2, J26.2, J27.2, J29.4, J30.4, JP42.2, JP43.2, JP44.2, JP45.2, PWR3.2
- net 3.3V5: now also ADR15.2, ADR16.2, ADR17.2, I2C5.2, INT5.2, J41.2, J42.2, J44.4, J45.1, J46.4, J48.2, PWR5.2; no longer 3V6.2, J31.2, J32.2, J33.2, J35.4, J36.4, JP50.2, JP51.2, JP52.2, JP53.2, JP54.2
- net 3.3V6: now also ADR18.2, ADR19.2, ADR20.2, I2C6.2, INT6.2, J49.2, J50.2, J52.4, J53.1, J54.4, J56.2, PWR6.2; no longer 3V7.2, J37.2, J38.2, J39.2, J41.4, J42.4, JP59.2, JP60.2, JP61.2, JP62.2, JP63.2
- net 3.3V7: now also ADR21.2, ADR22.2, ADR23.2, I2C7.2, INT7.2, J57.2, J58.2, J60.4, J61.1, J62.4, J64.2, PWR7.2; no longer 3V8.2, J43.2, J44.2, J45.2, J47.4, J48.4, JP68.2, JP69.2, JP70.2, JP71.2, JP72.2
- net 3.3V8: now also ADR24.2, ADR25.2, ADR26.2, I2C8.2, INT8.2, J65.2, J66.2, J68.4, J69.1, J70.4, J72.2, PWR8.2; no longer I2C6.2, J49.2, J50.2, J51.2, J53.4, J54.4, JP78.2, JP79.2, JP80.2, JP81.2, PWR6.2
- net GND: now also J1.4, J5.4, J8.1, J9.1; no longer J3.1, J5.1
- net GND1: now also J10.1, J11.4, J13.4, J14.1, J16.1, J3.1; no longer J11.1, J7.1, J8.1, J9.1
- net GND2: now also J19.4, J20.1, J21.4, J22.1, J24.1; no longer J13.1, J14.1, J15.1
- net GND3: now also J25.1, J26.1, J27.4, J28.1, J29.4, J30.1, J32.1; no longer J19.1, J20.1, J21.1, J23.1, J24.1
- net GND4: now also J33.1, J34.1, J35.4, J36.1, J37.4, J38.1, J40.1; no longer J25.1, J26.1, J27.1, J29.1, J30.1
- net GND5: now also J41.1, J42.1, J43.4, J44.1, J45.4, J46.1, J48.1; no longer J31.1, J32.1, J33.1, J35.1, J36.1
- net GND6: now also J49.1, J50.1, J51.4, J52.1, J53.4, J54.1, J56.1; no longer J37.1, J38.1, J39.1, J41.1, J42.1
- net GND7: now also J57.1, J58.1, J59.4, J60.1, J61.4, J62.1, J64.1; no longer J43.1, J44.1, J45.1, J47.1, J48.1
- net GND8: now also J65.1, J66.1, J67.4, J68.1, J69.4, J70.1, J72.1; no longer J49.1, J50.1, J51.1, J53.1, J54.1
- net N$1: now also INT.1; no longer JP8.1
- net N$10: now also INT3.1; no longer JP33.1
- net N$12: now also PWR3.1; no longer 3V4.1
- net N$13: now also INT4.1; no longer JP42.1
- net N$15: now also PWR4.1; no longer PWR3.1
- net N$16: now also INT5.1; no longer JP51.1
- net N$18: now also PWR5.1; no longer 3V6.1
- net N$19: now also INT6.1; no longer JP60.1
- net N$21: now also PWR6.1; no longer 3V7.1
- net N$22: now also INT7.1; no longer JP69.1
- net N$24: now also PWR7.1; no longer 3V8.1
- net N$25: now also INT8.1; no longer JP78.1
- net N$27: now also PWR8.1; no longer PWR6.1
- net N$4: now also INT1.1; no longer JP15.1
- net N$6: now also PWR1.1; no longer 3V1.1
- net N$7: now also INT2.1; no longer JP24.1
- net N$9: now also PWR2.1; no longer 3V2.1
- net P10: now also J14.3, U1.7; no longer J18.3, U2.7
- net P11: now also J11.3, U1.5; no longer J17.3, U2.5
- net P12: now also J13.2, U1.9; no longer J23.2, U4.4
- net P13: now also J13.3, U1.10; no longer J24.2, U4.6
- net P14: now also J12.2, U1.11; no longer J24.3, U4.7
- net P15: now also J12.3, U1.12; no longer J23.3, U4.5
- net P16: now also J19.2, U2.4; no longer J29.2, U5.4
- net P17: now also J22.2, U2.6; no longer J30.2, U5.6
- net P18: now also J22.3, U2.7; no longer J30.3, U5.7
- net P19: now also J19.3, U2.5; no longer J29.3, U5.5
- net P2: now also J8.2; no longer J6.2
- net P20: now also J21.2, U2.9; no longer J35.2, U6.4
- net P21: now also J21.3, U2.10; no longer J36.2, U6.6
- net P22: now also J20.2, U2.11; no longer J36.3, U6.7
- net P23: now also J20.3, U2.12; no longer J35.3, U6.5
- net P24: now also J27.2, U4.4; no longer J41.2, U7.4
- net P25: now also J30.2, U4.6; no longer J42.2, U7.6
- net P26: now also J30.3, U4.7; no longer J42.3, U7.7
- net P27: now also J27.3, U4.5; no longer J41.3, U7.5
- net P28: now also J29.2, U4.9; no longer J47.2, U8.4
- net P29: now also J29.3, U4.10; no longer J48.2, U8.6
- net P3: now also J8.3; no longer J6.3
- net P30: now also J28.2, U4.11; no longer J48.3, U8.7
- net P31: now also J28.3, U4.12; no longer J47.3, U8.5
- net P32: now also J35.2, U5.4; no longer J53.2, U9.4
- net P33: now also J38.2, U5.6; no longer J54.2, U9.6
- net P34: now also J38.3, U5.7; no longer J54.3, U9.7
- net P35: now also J35.3, U5.5; no longer J53.3, U9.5
- net P36: now also J37.2, U5.9; no longer J59.2, U10.4
- net P37: now also J37.3, U5.10; no longer J60.2, U10.6
- net P38: now also J36.2, U5.11; no longer J60.3, U10.7
- net P39: now also J36.3, U5.12; no longer J59.3, U10.5
- net P4: now also J1.2, U3.9; no longer J11.2, U1.4
- net P40: now also J43.2, U6.4; no longer J65.2, U11.4
- net P41: now also J46.2, U6.6; no longer J66.2, U11.6
- net P42: now also J46.3, U6.7; no longer J66.3, U11.7
- net P43: now also J43.3, U6.5; no longer J65.3, U11.5
- net P44: now also J45.2, U6.9; no longer J71.2, U12.4
- net P45: now also J45.3, U6.10; no longer J72.2, U12.6
- net P46: now also J44.2, U6.11; no longer J72.3, U12.7
- net P47: now also J44.3, U6.12; no longer J71.3, U12.5
- net P48: now also J51.2, U7.4; no longer J77.2, U13.4
- net P49: now also J54.2, U7.6; no longer J78.2, U13.6
- net P5: now also J1.3, U3.10; no longer J12.2, U1.6
- net P50: now also J54.3, U7.7; no longer J78.3, U13.7
- net P51: now also J51.3, U7.5; no longer J77.3, U13.5
- net P52: now also J53.2, U7.9; no longer J83.2, U14.4
- net P53: now also J53.3, U7.10; no longer J84.2, U14.6
- net P54: now also J52.2, U7.11; no longer J84.3, U14.7
- net P55: now also J52.3, U7.12; no longer J83.3, U14.5
- net P56: now also J59.2, U8.4; no longer J89.2, U15.4
- net P57: now also J62.2, U8.6; no longer J90.2, U15.6
- net P58: now also J62.3, U8.7; no longer J90.3, U15.7
- net P59: now also J59.3, U8.5; no longer J89.3, U15.5
- net P6: now also J6.2, U3.11; no longer J12.3, U1.7
- net P60: now also J61.2, U8.9; no longer J95.2, U16.4
- net P61: now also J61.3, U8.10; no longer J96.2, U16.6
- net P62: now also J60.2, U8.11; no longer J96.3, U16.7
- net P63: now also J60.3, U8.12; no longer J95.3, U16.5
- net P7: now also J6.3, U3.12; no longer J11.3, U1.5
- net P8: now also J11.2, U1.4; no longer J17.2, U2.4
- net P9: now also J14.2, U1.6; no longer J18.2, U2.6
- net SCL: now also J9.4; no longer J3.4
- net SCL1: now also J10.4, J16.4, J3.4; no longer J7.4, J8.4, J9.4
- net SCL2: now also J17.4, J18.4, J24.4; no longer J13.4, J14.4, J15.4
- net SCL3: now also J25.4, J26.4, J32.4; no longer J19.4, J20.4, J21.4
- net SCL4: now also J33.4, J34.4, J40.4; no longer J25.4, J26.4, J27.4
- net SCL5: now also J41.4, J42.4, J48.4; no longer J31.4, J32.4, J33.4
- net SCL6: now also J49.4, J50.4, J56.4; no longer J37.4, J38.4, J39.4
- net SCL7: now also J57.4, J58.4, J64.4; no longer J43.4, J44.4, J45.4
- net SCL8: now also J65.4, J66.4, J72.4; no longer J49.4, J50.4, J51.4
- net SCL_PU1: now also I2C.1; no longer JP10.1
- net SCL_PU2: now also I2C1.1; no longer JP14.1
- net SCL_PU3: now also I2C2.1; no longer JP23.1
- net SCL_PU4: now also I2C3.1; no longer JP32.1
- net SCL_PU5: now also I2C4.1; no longer I2C3.1
- net SCL_PU6: now also I2C5.1; no longer JP50.1
- net SCL_PU7: now also I2C6.1; no longer JP59.1
- net SCL_PU8: now also I2C7.1; no longer JP68.1
- net SCL_PU9: now also I2C8.1; no longer I2C6.1
- net SDA: now also J9.3; no longer J3.3
- net SDA1: now also J10.3, J16.3, J3.3; no longer J7.3, J8.3, J9.3
- net SDA2: now also J17.3, J18.3, J24.3; no longer J13.3, J14.3, J15.3
- net SDA3: now also J25.3, J26.3, J32.3; no longer J19.3, J20.3, J21.3
- net SDA4: now also J33.3, J34.3, J40.3; no longer J25.3, J26.3, J27.3
- net SDA5: now also J41.3, J42.3, J48.3; no longer J31.3, J32.3, J33.3
- net SDA6: now also J49.3, J50.3, J56.3; no longer J37.3, J38.3, J39.3
- net SDA7: now also J57.3, J58.3, J64.3; no longer J43.3, J44.3, J45.3
- net SDA8: now also J65.3, J66.3, J72.3; no longer J49.3, J50.3, J51.3
- net SDA_PU1: now also I2C.3; no longer JP10.3
- net SDA_PU2: now also I2C1.3; no longer JP14.3
- net SDA_PU3: now also I2C2.3; no longer JP23.3
- net SDA_PU4: now also I2C3.3; no longer JP32.3
- net SDA_PU5: now also I2C4.3; no longer I2C3.3
- net SDA_PU6: now also I2C5.3; no longer JP50.3
- net SDA_PU7: now also I2C6.3; no longer JP59.3
- net SDA_PU8: now also I2C7.3; no longer JP68.3
- net SDA_PU9: now also I2C8.3; no longer I2C6.3
Routing:
- net 3.3V9: track 97.8 -> 0.00 mm, vias 2 -> 0
- net 3.3V13: track 97.8 -> 0.00 mm, vias 2 -> 0
- net 3.3V11: track 97.8 -> 0.00 mm, vias 2 -> 0
- net 3.3V10: track 97.8 -> 0.00 mm, vias 2 -> 0
- net 3.3V14: track 97.8 -> 0.00 mm, vias 2 -> 0
- net 3.3V15: track 97.8 -> 0.00 mm, vias 2 -> 0
- net 3.3V12: track 97.8 -> 0.00 mm, vias 2 -> 0
- net 3.3V3: track 97.8 -> 157.5 mm, vias 2 -> 3
- net 3.3V5: track 97.8 -> 157.5 mm, vias 2 -> 3
- net 3.3V8: track 97.8 -> 157.5 mm, vias 2 -> 3
- net 3.3V1: track 97.8 -> 157.5 mm, vias 2 -> 3
- net 3.3V: track 97.8 -> 157.5 mm, vias 2 -> 3
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- removed copper zone on layer 1, net GND10
- removed copper zone on layer 16, net GND10
- removed copper zone on layer 1, net GND11
- removed copper zone on layer 16, net GND11
- removed copper zone on layer 1, net GND12
- removed copper zone on layer 16, net GND12
- removed copper zone on layer 1, net GND13
- removed copper zone on layer 16, net GND13
- removed copper zone on layer 1, net GND14
- removed copper zone on layer 16, net GND14
- removed copper zone on layer 1, net GND15
- removed copper zone on layer 16, net GND15
- removed copper zone on layer 1, net GND9
- removed copper zone on layer 16, net GND9
Other:
- board size 174 x 174 mm -> 204 x 135.4 mm
- board text added: "Andy England"
- board text added: "Kevin Kuwata"
- board text added: "v10"
